File: template/template.kicad_pcb (KiCad board)
At the start: 2 copper layers, 5 parts

Commit message: template update
Parts:
- removed LOGO1: Author Details, logos:template-details
- removed LOGO2: OSHW_FMask, logos:OSHW_Logo_3.6x3.6_F.Mask
- removed LOGO3: Board-Title, logos:board-title
- removed LOGO4: Logo, logos:OSHW-Logo2_9.8x8mm_Mask
- removed LOGO5: 4-Layer-Check, logos:4-layer-check
