File: template/template.sch (KiCad schematic (older format))
At the start: 5 parts

Commit message: template update
Parts:
- removed LOGO1: Author Details, logos:template-details, symbol Mechanical:MountingHole
- removed LOGO2: OSHW_FMask, logos:OSHW_Logo_3.6x3.6_F.Mask, symbol Graphic:Logo_Open_Hardware_Small
- removed LOGO3: Board-Title, logos:board-title, symbol Mechanical:MountingHole
- removed LOGO4: Logo, logos:OSHW-Logo2_9.8x8mm_Mask, symbol Mechanical:MountingHole
- removed LOGO5: 4-Layer-Check, logos:4-layer-check, symbol Mechanical:MountingHole
Other:
- note removed: "Logos / Markings"
Changed lines of the file:
@@
 Comment4 ""
 $EndDescr
-$Comp
-L Graphic:Logo_Open_Hardware_Small LOGO2
-U 1 1 5E2031A4
-P 6600 7500
-F 0 "LOGO2" H 6600 7886 50  0000 C CNN
-F 1 "OSHW_FMask" H 6600 7795 50  0000 C CNN
-F 2 "logos:OSHW_Logo_3.6x3.6_F.Mask" H 6600 7500 50  0001 C CNN
-F 3 "~" H 6600 7500 50  0001 C CNN
-	1    6600 7500
-	0    1    1    0
-$EndComp
-$Comp
-L Mechanical:MountingHole LOGO1
-U 1 1 5E204886
-P 6050 7200
-F 0 "LOGO1" H 6050 7437 50  0000 C CNN
-F 1 "Author Details" H 6050 7346 50  0000 C CNN
-F 2 "logos:template-details" H 6050 7200 50  0001 C CNN
-F 3 "~" H 6050 7200 50  0001 C CNN
-	1    6050 7200
-	1    0    0    -1
-$EndComp
-$Comp
-L Mechanical:MountingHole LOGO5
-U 1 1 5E2051A0
-P 6050 7650
-F 0 "LOGO5" H 6050 7887 50  0000 C CNN
-F 1 "4-Layer-Check" H 6050 7796 50  0000 C CNN
-F 2 "logos:4-layer-check" H 6050 7650 50  0001 C CNN
-F 3 "~" H 6050 7650 50  0001 C CNN
-	1    6050 7650
-	1    0    0    -1
-$EndComp
-Text Notes 5350 6850 0    100  ~ 0
-Logos / Markings
-$Comp
-L Mechanical:MountingHole LOGO4
-U 1 1 5E2057DD
-P 5400 7650
-F 0 "LOGO4" H 5400 7887 50  0000 C CNN
-F 1 "Logo" H 5400 7796 50  0000 C CNN
-F 2 "logos:OSHW-Logo2_9.8x8mm_Mask" H 5400 7650 50  0001 C CNN
-F 3 "~" H 5400 7650 50  0001 C CNN
-	1    5400 7650
-	1    0    0    -1
-$EndComp
-$Comp
-L Mechanical:MountingHole LOGO3
-U 1 1 5E205A57
-P 5400 7200
-F 0 "LOGO3" H 5400 7437 50  0000 C CNN
-F 1 "Board-Title" H 5400 7346 50  0000 C CNN
-F 2 "logos:board-title" H 5400 7200 50  0001 C CNN
-F 3 "~" H 5400 7200 50  0001 C CNN
-	1    5400 7200
-	1    0    0    -1
-$EndComp
 $EndSCHEMATC
